Commit message: controlling

File: description/robot.urdf.xacro (robot description, xacro)
@@ -5,3 +5,5 @@
     <!-- including robot core structure -->
     <xacro:include filename= 'robot_core.xacro' />
+    <!-- including robot gazebo control -->
+    <xacro:include filename= 'gazebo_control.xacro' />
 </robot>

File: description/robot_core.xacro (robot description, xacro)
@@ -41,4 +41,7 @@
         </xacro:inertial_box>
     </link>
+    <gazebo reference="chassis">
+        <material> Gazebo/White </material>
+    </gazebo>
     <!-- LEFT WHEEL -->
     <joint name="left_wheel_joint" type="continuous">
@@ -56,7 +59,6 @@
         </visual>
         <collision>
-            <origin xyz="0.15 0 0.075" rpy="0 0 0"/>
             <geometry>
-                <box size="0.3 0.3 0.15"/>
+                <cylinder length="0.04" radius="0.05" />/>
             </geometry>
         </collision>
@@ -65,4 +67,7 @@
         </xacro:inertial_cylinder>
     </link>
+    <gazebo reference="left_wheel">
+        <material> Gazebo/Blue </material>
+    </gazebo>
     <!-- RIGHT WHEEL -->
     <joint name="right_wheel_joint" type="continuous">
@@ -80,7 +85,6 @@
         </visual>
         <collision>
-            <origin xyz="0.15 0 0.075" rpy="0 0 0"/>
             <geometry>
-                <box size="0.3 0.3 0.15"/>
+                <cylinder length="0.04" radius="0.05" />/>
             </geometry>
         </collision>
@@ -89,4 +93,7 @@
         </xacro:inertial_cylinder>
     </link>
+    <gazebo reference="right_wheel">
+        <material> Gazebo/Blue </material>
+    </gazebo>
     <!-- CASTER WHEEL -->
     <joint name="caster_wheel_joint" type="fixed">
@@ -103,7 +110,6 @@
         </visual>
         <collision>
-            <origin xyz="0.15 0 0.075" rpy="0 0 0"/>
             <geometry>
-                <box size="0.3 0.3 0.15"/>
+                <sphere radius="0.05" />
             </geometry>
         </collision>
@@ -112,3 +118,9 @@
         </xacro:inertial_sphere>
     </link>
+    <gazebo reference="caster_wheel">
+        <material> Gazebo/Black </material>
+        <!-- reducing frictions -->
+        <mu1 value="0.001"/>
+        <mu2 value="0.001"/>
+    </gazebo>
 </robot>

Commit message: adding cameras lidar and control

File: description/robot.urdf.xacro (robot description, xacro)
@@ -5,5 +5,15 @@
     <!-- including robot core structure -->
     <xacro:include filename= 'robot_core.xacro' />
+    <!-- need to comment the control not used -->
     <!-- including robot gazebo control -->
-    <xacro:include filename= 'gazebo_control.xacro' />
+    <!--<xacro:include filename= 'gazebo_control.xacro' />-->
+    <!-- including ros2_control -->
+    <xacro:include filename= 'ros2_control.xacro' />
+    <!-- including lidar in gazebo -->
+    <xacro:include filename= 'lidar.xacro' />
+    <!-- need to comment the camera not used -->
+    <!-- including camera in gazebo -->
+    <!--<xacro:include filename= 'camera.xacro' />-->
+    <!-- including depth camera in gazebo -->
+    <xacro:include filename= 'depth_camera.xacro' />
 </robot>

File: description/robot_core.xacro (robot description, xacro)
@@ -14,4 +14,7 @@
     <material name="black">
         <color rgba="0 0 0 1"/>
+    </material>
+    <material name="red">
+        <color rgba="1 0 0 1"/>
     </material>
     <!-- BASE LINK & CHASSIS -->
