Commit message: adding teleop with joystick and other mods

File: description/camera.xacro (robot description, xacro)
@@ -4,5 +4,6 @@
         <parent link="chassis"/>
         <child link="camera_link"/>
-        <origin xyz="0.305 0 0.08" rpy="0 0 0"/>
+        <!--<origin xyz="0.305 0 0.08" rpy="0 0 0"/> -->
+        <origin xyz="0.4 0 0.08" rpy="0 0 0"/>
     </joint>
     <link name="camera_link">

File: description/depth_camera.xacro (robot description, xacro)
@@ -4,5 +4,6 @@
         <parent link="chassis"/>
         <child link="camera_link"/>
-        <origin xyz="0.305 0 0.08" rpy="0 0 0"/>
+        <!--<origin xyz="0.305 0 0.08" rpy="0 0 0"/> -->
+        <origin xyz="0.4 0 0.08" rpy="0 0 0"/>
     </joint>
     <link name="camera_link">

File: description/lidar.xacro (robot description, xacro)
@@ -4,5 +4,6 @@
         <parent link="chassis"/>
         <child link="laser_frame"/>
-        <origin xyz="0.1 0 0.175" rpy="0 0 0"/>
+        <!--<origin xyz="0.1 0 0.175" rpy="0 0 0"/> -->
+        <origin xyz="0.1 0 0.14" rpy="0 0 0"/>
     </joint>
     <link name="laser_frame">

File: description/robot.urdf.xacro (robot description, xacro)
@@ -3,4 +3,6 @@
     <!-- Example link -->
     <!-- <link name="base_link"></link> -->
+    <!-- to pass from gazebo_control to ros2_control-->
+    <xacro:arg name="use_ros2_control" default="true"/>
     <!-- including robot core structure -->
     <xacro:include filename= 'robot_core.xacro' />
@@ -9,11 +11,18 @@
     <!--<xacro:include filename= 'gazebo_control.xacro' />-->
     <!-- including ros2_control -->
-    <xacro:include filename= 'ros2_control.xacro' />
+    <!--<xacro:include filename= 'ros2_control.xacro' />-->
+    <!-- PROBLEM 3 -->
+    <xacro:if value="$(arg use_ros2_control)">
+        <xacro:include filename="ros2_control.xacro" />
+    </xacro:if>
+    <xacro:unless value="$(arg use_ros2_control)">
+        <xacro:include filename="gazebo_control.xacro" />
+    </xacro:unless>
     <!-- including lidar in gazebo -->
     <xacro:include filename= 'lidar.xacro' />
     <!-- need to comment the camera not used -->
     <!-- including camera in gazebo -->
-    <!--<xacro:include filename= 'camera.xacro' />-->
+    <xacro:include filename= 'camera.xacro' />
     <!-- including depth camera in gazebo -->
-    <xacro:include filename= 'depth_camera.xacro' />
+    <!--<xacro:include filename= 'depth_camera.xacro' />-->
 </robot>

File: description/robot_core.xacro (robot description, xacro)
@@ -30,5 +30,6 @@
             <origin xyz="0.15 0 0.075" rpy="0 0 0"/>
             <geometry>
-                <box size="0.3 0.3 0.15"/>
+                <!-- <box size="0.3 0.3 0.15"/> -->
+                <cylinder length="0.1" radius="0.25" />/>
             </geometry>
             <material name="white"/>
@@ -37,5 +38,6 @@
             <origin xyz="0.15 0 0.075" rpy="0 0 0"/>
             <geometry>
-                <box size="0.3 0.3 0.15"/>
+                <!--<box size="0.3 0.3 0.15"/>-->
+                <cylinder length="0.1" radius="0.25" />/>
             </geometry>
         </collision>
@@ -61,7 +63,9 @@
             <material name="blue"/>
         </visual>
+        <!--PROBLEM 2 wheel drift solved replacing cylinder with sphere-->
         <collision>
             <geometry>
-                <cylinder length="0.04" radius="0.05" />/>
+                <!--<cylinder length="0.04" radius="0.05" />/>-->
+                <sphere radius="0.05" />/>
             </geometry>
         </collision>
@@ -89,5 +93,6 @@
         <collision>
             <geometry>
-                <cylinder length="0.04" radius="0.05" />/>
+                <!--<cylinder length="0.04" radius="0.05" />/>-->
+                <sphere radius="0.05" />/>
             </geometry>
         </collision>

Commit message: final results

File: description/camera.xacro (robot description, xacro)
@@ -5,5 +5,5 @@
         <child link="camera_link"/>
         <!--<origin xyz="0.305 0 0.08" rpy="0 0 0"/> -->
-        <origin xyz="0.4 0 0.08" rpy="0 0 0"/>
+        <origin xyz="0.4 0 0.18" rpy="0 0 0"/>
     </joint>
     <link name="camera_link">

File: description/depth_camera.xacro (robot description, xacro)
@@ -5,5 +5,5 @@
         <child link="camera_link"/>
         <!--<origin xyz="0.305 0 0.08" rpy="0 0 0"/> -->
-        <origin xyz="0.4 0 0.08" rpy="0 0 0"/>
+        <origin xyz="0.4 0 0.18" rpy="0 0 0"/>
     </joint>
     <link name="camera_link">

File: description/lidar.xacro (robot description, xacro)
@@ -4,6 +4,7 @@
         <parent link="chassis"/>
         <child link="laser_frame"/>
+        <!--<origin xyz="0.1 0 0.14" rpy="0 0 0"/>-->
         <!--<origin xyz="0.1 0 0.175" rpy="0 0 0"/> -->
-        <origin xyz="0.1 0 0.14" rpy="0 0 0"/>
+        <origin xyz="0.1 0 0.55" rpy="0 0 0"/>
     </joint>
     <link name="laser_frame">

File: description/robot_core.xacro (robot description, xacro)
@@ -37,21 +37,26 @@
     <link name="chassis">
         <visual>
-            <origin xyz="0.15 0 0.075" rpy="0 0 0"/>
+            <!--<origin xyz="0.15 0 0.075" rpy="0 0 0"/>-->
+            <origin xyz="0.15 0 0.275" rpy="0 0 0"/>
             <geometry>
                 <!-- <box size="0.3 0.3 0.15"/> -->
-                <cylinder length="0.1" radius="0.25" />/>
+                <!--<cylinder length="0.1" radius="0.25" />/>-->
+                <cylinder length="0.5" radius="0.25" />/>
             </geometry>
             <material name="white"/>
         </visual>
         <collision>
-            <origin xyz="0.15 0 0.075" rpy="0 0 0"/>
+            <origin xyz="0.15 0 0.275" rpy="0 0 0"/>
             <geometry>
                 <!--<box size="0.3 0.3 0.15"/>-->
-                <cylinder length="0.1" radius="0.25" />/>
+                <cylinder length="0.5" radius="0.25" />/>
             </geometry>
         </collision>
-        <xacro:inertial_box mass="0.5" x="0.3" y="0.3" z="0.15">
+        <!--<xacro:inertial_box mass="0.5" x="0.3" y="0.3" z="0.15">
             <origin xyz="0.15 0 0.075" rpy="0 0 0"/>
-        </xacro:inertial_box>
+        </xacro:inertial_box>-->
+        <xacro:inertial_cylinder mass="0.5" length="0.5" radius="0.25">
+            <origin xyz="0.15 0 0.275" rpy="0 0 0"/>
+        </xacro:inertial_cylinder>
     </link>
     <gazebo reference="chassis">
